Commit message: fixes

File: hege_ws/src/hege_description/urdf/hege.urdf.xacro (robot description, xacro)
@@ -27,5 +27,4 @@
       <mu1>${wheel_mu_longitudinal}</mu1>
       <mu2>${wheel_mu_lateral}</mu2>
-      <fdir1>1 0 0</fdir1>
       <kp>10000000.0</kp>
       <kd>10000.0</kd>
@@ -53,5 +52,5 @@
     <parent link="base_footprint"/>
     <child link="base_link"/>
-    <origin xyz="0 0 ${base_height}" rpy="0 0 0"/>
+    <origin xyz="0.95 0 ${base_height}" rpy="0 0 0"/>
   </joint>
   <xacro:macro name="rear_wheel" params="side y_sign">
@@ -142,8 +141,26 @@
       <topic>/gps/fix</topic>
       <navsat><position_sensing>
-        <horizontal><noise type="gaussian"><mean>0</mean><stddev>${gps_horizontal_stddev}</stddev></noise></horizontal>
-        <vertical><noise type="gaussian"><mean>0</mean><stddev>${gps_vertical_stddev}</stddev></noise></vertical>
+        <!-- gz-sensors8 NavSatSensor::Update applies this value to
+             Latitude().Degree() and Longitude().Degree(). A 2.0 metre target
+             therefore needs about 1.8e-5 degrees, not the literal value 2.0. -->
+        <horizontal><noise type="gaussian"><mean>0</mean><stddev>${gps_horizontal_stddev_m/metres_per_latitude_degree}</stddev></noise></horizontal>
+        <vertical><noise type="gaussian"><mean>0</mean><stddev>${gps_vertical_stddev_m}</stddev></noise></vertical>
       </position_sensing></navsat>
     </sensor>
+  </gazebo>
+  <!-- Noise-free Gazebo truth for evaluation only. This topic must never be
+       fused into the GPS navigation estimator. Keeping it under /hege avoids
+       PX4's default odometry topic names when the SITL path is added later. -->
+  <gazebo>
+    <plugin filename="gz-sim-odometry-publisher-system"
+            name="gz::sim::systems::OdometryPublisher">
+      <odom_frame>world</odom_frame>
+      <robot_base_frame>base_footprint</robot_base_frame>
+      <dimensions>3</dimensions>
+      <odom_publish_frequency>50</odom_publish_frequency>
+      <odom_topic>/hege/ground_truth/odom</odom_topic>
+      <odom_covariance_topic>/hege/ground_truth/odom_with_covariance</odom_covariance_topic>
+      <tf_topic>/hege/ground_truth/pose</tf_topic>
+    </plugin>
   </gazebo>
   <ros2_control name="HegeGazeboSystem" type="system">

File: hege_ws/src/hege_description/urdf/hege_parameters.xacro (robot description, xacro)
@@ -50,10 +50,15 @@
   <xacro:property name="max_linear_speed" value="0.30"/>
   <xacro:property name="rear_wheel_speed_limit" value="${max_linear_speed/rear_wheel_radius}"/>
-  <xacro:property name="wheel_mu_longitudinal" value="0.80"/>
-  <xacro:property name="wheel_mu_lateral" value="1.00"/>
+  <xacro:property name="wheel_mu_longitudinal" value="0.8"/>
+  <xacro:property name="wheel_mu_lateral" value="0.8"/>
   <xacro:property name="wheel_slip" value="0.02"/>
-  <!-- Sensor model: standalone GNSS and a typical MEMS IMU starting point. -->
-  <xacro:property name="gps_horizontal_stddev" value="2.0"/>
-  <xacro:property name="gps_vertical_stddev" value="4.0"/>
+  <!-- Sensor model: standalone GNSS and a typical MEMS IMU starting point.
+       gz-sensors8 applies horizontal NavSat noise directly to latitude and
+       longitude expressed in DEGREES, while vertical noise is in metres.
+       Keep the human-facing horizontal parameter in metres and convert it in
+       hege.urdf.xacro. Never feed a metre value directly to <horizontal>. -->
+  <xacro:property name="gps_horizontal_stddev_m" value="2.0"/>
+  <xacro:property name="gps_vertical_stddev_m" value="4.0"/>
+  <xacro:property name="metres_per_latitude_degree" value="111195.0"/>
   <xacro:property name="imu_gyro_noise" value="2.0e-4"/>
   <xacro:property name="imu_accel_noise" value="1.7e-2"/>
